File: AMG8833 Deck Board/TA_v2_Deck.brd (EAGLE design)
At the start: 29.5 x 31 mm, 10 parts, among them U2 3.3V

Commit message: Fix Board Design
Routing:
- net GND: track 79.9 -> 82.2 mm
- net VBAT: track 7.87 -> 9.00 mm
Other:
- outline, holes or cut-outs redrawn
Changed lines of the file:
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@@
 <setting verticaltext="up"/>
 </settings>
-<grid distance="0.5" unitdist="mm" unit="mm" style="lines" multiple="1" display="yes" altdistance="5" altunitdist="mil" altunit="mil"/>
+<grid distance="1" unitdist="mil" unit="mil" style="lines" multiple="1" display="yes" altdistance="5" altunitdist="mil" altunit="mil"/>
 <layers>
 <layer number="1" name="Top" color="4" fill="1" visible="yes" active="yes"/>
@@
 <layer number="25" name="tNames" color="7" fill="1" visible="yes" active="yes"/>
 <layer number="26" name="bNames" color="7" fill="1" visible="yes" active="yes"/>
-<layer number="27" name="tValues" color="7" fill="1" visible="yes" active="yes"/>
-<layer number="28" name="bValues" color="7" fill="1" visible="yes" active="yes"/>
+<layer number="27" name="tValues" color="7" fill="1" visible="no" active="yes"/>
+<layer number="28" name="bValues" color="7" fill="1" visible="no" active="yes"/>
 <layer number="29" name="tStop" color="7" fill="3" visible="no" active="yes"/>
 <layer number="30" name="bStop" color="7" fill="6" visible="no" active="yes"/>
@@
 <layer number="44" name="Drills" color="7" fill="1" visible="no" active="yes"/>
 <layer number="45" name="Holes" color="7" fill="1" visible="no" active="yes"/>
-<layer number="46" name="Milling" color="3" fill="1" visible="yes" active="yes"/>
-<layer number="47" name="Measures" color="7" fill="1" visible="yes" active="yes"/>
+<layer number="46" name="Milling" color="3" fill="1" visible="no" active="yes"/>
+<layer number="47" name="Measures" color="7" fill="1" visible="no" active="yes"/>
 <layer number="48" name="Document" color="7" fill="1" visible="no" active="yes"/>
 <layer number="49" name="Reference" color="7" fill="1" visible="no" active="yes"/>
@@
 <wire x1="0" y1="25.5" x2="0" y2="6.5" width="0" layer="20"/>
 <wire x1="29.5" y1="6.5" x2="29.5" y2="25.5" width="0" layer="20"/>
-<dimension x1="1" y1="6.5" x2="28.5" y2="6.5" x3="14.75" y3="-10.9" textsize="1.778" layer="47"/>
 <dimension x1="1" y1="6.5" x2="6.4" y2="6.5" x3="3.7" y3="-3.1" textsize="1.778" layer="47"/>
 <dimension x1="3.7" y1="16" x2="25.8" y2="16" x3="14.75" y3="-7" textsize="1.778" layer="47"/>
@@
 <wire x1="23.5" y1="30.5" x2="6" y2="30.5" width="0.254" layer="21"/>
 <wire x1="1" y1="25.5" x2="6" y2="30.5" width="0.254" layer="21"/>
-<circle x="5.3" y="26.9" radius="0.70710625" width="0.254" layer="21"/>
-<circle x="5.3" y="26.9" radius="0.14141875" width="0.254" layer="21"/>
-<wire x1="5.3" y1="26.9" x2="5.3" y2="28.7" width="0.254" layer="21"/>
-<wire x1="5.3" y1="28.7" x2="5" y2="28.2" width="0.254" layer="21"/>
-<wire x1="5.3" y1="28.7" x2="5.6" y2="28.2" width="0.254" layer="21"/>
+<circle x="5.3" y="27.154" radius="0.889" width="0.254" layer="21"/>
+<wire x1="5.3" y1="27.154" x2="5.2746" y2="29.208" width="0.3048" layer="21"/>
+<wire x1="5.2746" y1="29.208" x2="4.873" y2="28.6826" width="0.4064" layer="21"/>
+<wire x1="5.2746" y1="29.208" x2="5.7016" y2="28.6826" width="0.4064" layer="21"/>
 <rectangle x1="8.652" y1="13.724" x2="21.098" y2="18.804" layer="41"/>
-<rectangle x1="8.652" y1="13.724" x2="21.098" y2="18.804" layer="42"/>
 <text x="14.494" y="29.218" size="0.6096" layer="25" distance="25" align="center">ESP32-AMG8833 Deck
 Made by Egar</text>
@@
 <wire x1="5.5" y1="31" x2="0" y2="25.5" width="0.0762" layer="20"/>
 <wire x1="24" y1="31" x2="29.5" y2="25.5" width="0.0762" layer="20"/>
+<wire x1="8.8" y1="18.6" x2="21.2" y2="18.6" width="0.0762" layer="20"/>
+<wire x1="21.2" y1="18.6" x2="21.2" y2="13.6" width="0.0762" layer="20"/>
+<wire x1="21.2" y1="13.6" x2="8.8" y2="13.6" width="0.0762" layer="20"/>
+<wire x1="8.8" y1="13.6" x2="8.8" y2="18.6" width="0.0762" layer="20"/>
+<dimension x1="6.5" y1="0" x2="6.5" y2="31" x3="-2.5" y3="15.5" textsize="1.778" layer="47"/>
+<dimension x1="0" y1="6.5" x2="29.5" y2="6.5" x3="14.75" y3="-11" textsize="1.778" layer="47"/>
+<wire x1="4.953" y1="26.7716" x2="5.6896" y2="27.5082" width="0.3048" layer="21"/>
+<wire x1="4.9276" y1="27.5082" x2="5.6896" y2="26.7716" width="0.3048" layer="21"/>
 </plain>
 <attributes>
@@
 <contactref element="U$2" pad="A"/>
 <via x="23.8826" y="4.8294" extent="1-16" drill="0.35"/>
-<wire x1="22.622" y1="8.644" x2="22.9743" y2="8.9963" width="0.6096" layer="1"/>
-<wire x1="22.622" y1="8.644" x2="22.622" y2="6.09" width="0.6096" layer="1"/>
-<wire x1="22.622" y1="6.09" x2="23.8826" y2="4.8294" width="0.6096" layer="1"/>
 <wire x1="23.8826" y1="4.8294" x2="23.3746" y2="4.3214" width="0.6096" layer="16"/>
 <wire x1="23.3746" y1="4.3214" x2="22.1046" y2="4.3214" width="0.6096" layer="16"/>
-<wire x1="22.9743" y1="8.9963" x2="24.017759375" y2="8.9963" width="0.6096" layer="1"/>
+<wire x1="27.617759375" y1="8.9963" x2="27.432" y2="8.810540625" width="0.4064" layer="1"/>
+<wire x1="23.8826" y1="4.8294" x2="24.6412" y2="5.588" width="0.6096" layer="1"/>
+<wire x1="27.617759375" y1="6.789759375" x2="27.617759375" y2="8.9963" width="0.6096" layer="1"/>
+<wire x1="24.6412" y1="5.588" x2="26.416" y2="5.588" width="0.6096" layer="1"/>
+<wire x1="26.416" y1="5.588" x2="27.617759375" y2="6.789759375" width="0.6096" layer="1"/>
 </signal>
 <signal name="VCC">
@@
 <contactref element="CON_BOARD" pad="5"/>
 <wire x1="18.119" y1="26.609" x2="18.22" y2="26.71" width="0.4064" layer="16"/>
-<wire x1="5.517759375" y1="6.9963" x2="5.604" y2="6.9963" width="0.4064" layer="1"/>
 <wire x1="15.516" y1="3.316" x2="15.516" y2="3.984" width="0.4064" layer="1"/>
 <wire x1="14.494" y1="2.294" x2="15.516" y2="3.316" width="0.4064" layer="1"/>
-<wire x1="5.604" y1="6.9963" x2="5.604" y2="4.834" width="0.4064" layer="1"/>
-<wire x1="5.604" y1="4.834" x2="6.112" y2="4.326" width="0.4064" layer="1"/>
 <via x="6.112" y="4.326" extent="1-16" drill="0.35"/>
 <wire x1="6.112" y1="4.326" x2="6.874" y2="5.088" width="0.4064" layer="16"/>
@@
 <vertex x="1.54" y="6.612"/>
 </polygon>
+<wire x1="2.132225" y1="6.9963" x2="1.887759375" y2="6.9963" width="0.4064" layer="1"/>
+<wire x1="4.5492" y1="5.8888" x2="3.239725" y2="5.8888" width="0.4064" layer="1"/>
+<wire x1="3.239725" y1="5.8888" x2="2.132225" y2="6.9963" width="0.4064" layer="1"/>
+<wire x1="6.112" y1="4.326" x2="4.5492" y2="5.8888" width="0.4064" layer="1"/>
 </signal>
 <signal name="EN">
