File: AMG8833 Deck Board/TA_v2_ESP.brd (EAGLE design)
At the start: 21 x 32.5 mm, 8 parts

Commit message: Fix Board Design
Parts:
- R1, R2: value 4.7k -> NC
Connections:
- net SCL: now also U$1.20; no longer U$1.21
- net SDA: now also U$1.21; no longer U$1.20
Routing:
- net SCL: track 9.27 -> 10.7 mm
- net SDA: track 8.89 -> 7.90 mm
Other:
- board size 21 x 32.5 mm -> 21 x 26.5 mm
Changed lines of the file:
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@@
 <setting verticaltext="up"/>
 </settings>
-<grid distance="50" unitdist="mil" unit="mil" style="lines" multiple="1" display="yes" altdistance="5" altunitdist="mil" altunit="mil"/>
+<grid distance="10" unitdist="mil" unit="mil" style="lines" multiple="1" display="yes" altdistance="5" altunitdist="mil" altunit="mil"/>
 <layers>
 <layer number="1" name="Top" color="4" fill="1" visible="yes" active="yes"/>
@@
 <plain>
 <wire x1="0" y1="0" x2="20.98" y2="0" width="0" layer="20"/>
-<wire x1="20.98" y1="0" x2="20.98" y2="32.5" width="0" layer="20"/>
-<wire x1="20.98" y1="32.5" x2="0" y2="32.5" width="0" layer="20"/>
-<wire x1="0" y1="32.5" x2="0" y2="0" width="0" layer="20"/>
-<dimension x1="-0.02" y1="0" x2="20.98" y2="0" x3="10.48" y3="-6.38" textsize="1.778" layer="47"/>
+<wire x1="20.98" y1="0" x2="20.98" y2="26.5" width="0" layer="20"/>
+<wire x1="20.98" y1="26.5" x2="0" y2="26.5" width="0" layer="20"/>
+<wire x1="0" y1="26.5" x2="0" y2="0" width="0" layer="20"/>
+<dimension x1="-0.02" y1="0" x2="20.98" y2="0" x3="10.48" y3="-4.856" textsize="1.778" layer="47"/>
 <text x="17.218" y="15.24" size="0.6096" layer="26" rot="MR270" align="center">LED</text>
 <text x="2.994" y="3.81" size="0.6096" layer="25" distance="25" align="center">ESP32
 Breakout
 Board</text>
+<dimension x1="0" y1="26.5" x2="0" y2="0" x3="-3.5" y3="13.25" textsize="1.778" layer="47"/>
 </plain>
 <attributes>
@@
 </autorouter>
 <elements>
-<element name="R1" library="rcl" library_urn="urn:adsk.eagle:library:334" package="R0603" package3d_urn="urn:adsk.eagle:package:23555/3" value="4.7k" x="6.796" y="15.044" smashed="yes" rot="MR270">
+<element name="R1" library="rcl" library_urn="urn:adsk.eagle:library:334" package="R0603" package3d_urn="urn:adsk.eagle:package:23555/3" value="NC" x="6.796" y="15.044" smashed="yes" rot="MR270">
 <attribute name="NAME" x="6.161" y="15.679" size="0.6096" layer="26" rot="MR270"/>
 <attribute name="POPULARITY" value="77" x="48.706" y="-28.136" size="1.778" layer="28" rot="MR270" display="off"/>
 <attribute name="SPICEPREFIX" value="R" x="48.706" y="-28.136" size="1.778" layer="28" rot="MR270" display="off"/>
 </element>
-<element name="R2" library="rcl" library_urn="urn:adsk.eagle:library:334" package="R0603" package3d_urn="urn:adsk.eagle:package:23555/3" value="4.7k" x="8.964" y="15.044" smashed="yes" rot="MR270">
+<element name="R2" library="rcl" library_urn="urn:adsk.eagle:library:334" package="R0603" package3d_urn="urn:adsk.eagle:package:23555/3" value="NC" x="8.964" y="15.044" smashed="yes" rot="MR270">
 <attribute name="NAME" x="8.329" y="15.679" size="0.6096" layer="26" rot="MR270"/>
 <attribute name="POPULARITY" value="77" x="57.224" y="-1.466" size="1.778" layer="28" rot="MR270" display="off"/>
@@
 <wire x1="17.634" y1="10.506" x2="16.456" y2="11.684" width="0.4064" layer="16"/>
 <polygon width="0.6096" layer="1" isolate="0.6096">
-<vertex x="0.962" y="22.86"/>
-<vertex x="20.012" y="22.86"/>
+<vertex x="0.962" y="22.36"/>
+<vertex x="20.012" y="22.36"/>
 <vertex x="20.012" y="0.508"/>
 <vertex x="0.962" y="0.508"/>
 </polygon>
 <polygon width="0.6096" layer="16" isolate="0.6096" rank="4">
-<vertex x="0.962" y="22.86"/>
-<vertex x="20.012" y="22.86"/>
+<vertex x="0.962" y="22.36"/>
+<vertex x="20.012" y="22.36"/>
 <vertex x="20.012" y="0.508"/>
 <vertex x="0.962" y="0.508"/>
@@
 <signal name="SDA">
 <contactref element="CON_ESP" pad="6"/>
-<contactref element="U$1" pad="20"/>
-<wire x1="11.411" y1="9.283" x2="11.46" y2="9.332" width="0.254" layer="1"/>
-<via x="12.554" y="11.43" extent="1-16" drill="0.35"/>
-<wire x1="11.85" y1="5.524" x2="11.85" y2="10.726" width="0.4064" layer="16"/>
-<wire x1="11.85" y1="10.726" x2="12.554" y2="11.43" width="0.4064" layer="16"/>
-<wire x1="12.554" y1="11.43" x2="11.411" y2="10.287" width="0.4064" layer="1"/>
-<wire x1="11.411" y1="10.287" x2="11.411" y2="9.283" width="0.4064" layer="1"/>
+<via x="13.054" y="10.914" extent="1-16" drill="0.35"/>
+<wire x1="11.85" y1="5.524" x2="13.374" y2="7.048" width="0.4064" layer="16"/>
+<wire x1="13.374" y1="10.594" x2="13.054" y2="10.914" width="0.4064" layer="16"/>
+<wire x1="13.374" y1="10.594" x2="13.374" y2="7.048" width="0.4064" layer="16"/>
+<contactref element="U$1" pad="21"/>
+<wire x1="13.054" y1="10.914" x2="13.46" y2="10.508" width="0.4064" layer="1"/>
+<wire x1="13.46" y1="10.508" x2="13.46" y2="9.332" width="0.4064" layer="1"/>
 </signal>
 <signal name="SCL">
 <contactref element="CON_ESP" pad="8"/>
-<contactref element="U$1" pad="21"/>
-<wire x1="13.46" y1="9.332" x2="13.46" y2="10.05" width="0.254" layer="1"/>
-<via x="14.586" y="11.43" extent="1-16" drill="0.35"/>
-<wire x1="14.39" y1="5.524" x2="14.39" y2="11.234" width="0.4064" layer="16"/>
-<wire x1="14.39" y1="11.234" x2="14.586" y2="11.43" width="0.4064" layer="16"/>
-<wire x1="14.586" y1="11.43" x2="13.46" y2="10.304" width="0.4064" layer="1"/>
-<wire x1="13.46" y1="10.304" x2="13.46" y2="9.332" width="0.4064" layer="1"/>
+<via x="14.324" y="11.422" extent="1-16" drill="0.35"/>
+<wire x1="14.39" y1="5.524" x2="14.39" y2="11.356" width="0.4064" layer="16"/>
+<wire x1="14.39" y1="11.356" x2="14.324" y2="11.422" width="0.4064" layer="16"/>
+<contactref element="U$1" pad="20"/>
+<wire x1="11.46" y1="9.332" x2="11.46" y2="10.698" width="0.4064" layer="1"/>
+<wire x1="11.46" y1="10.698" x2="12.446" y2="11.684" width="0.4064" layer="1"/>
+<wire x1="12.446" y1="11.684" x2="14.062" y2="11.684" width="0.4064" layer="1"/>
+<wire x1="14.062" y1="11.684" x2="14.324" y2="11.422" width="0.4064" layer="1"/>
 </signal>
 <signal name="N$7">
